Commit message: [first_robot_gazebo]rplidar urdf and dae files added

File: sim/first_robot_gazebo/definition/laser.urdf.xacro (robot description, xacro)
@@ -1,30 +1,60 @@
-<?xml version="1.0"?>
-<robot name="sensor_hokuyo" xmlns:xacro="http://ros.org/wiki/xacro">
-  <xacro:include filename="$(find turtlebot_description)/urdf/turtlebot_gazebo.urdf.xacro"/>
-  <xacro:include filename="$(find turtlebot_description)/urdf/turtlebot_properties.urdf.xacro"/>
-  <!-- Hokuyo 2D LIDAR -->
-  <xacro:macro name="sensor_hokuyo" params="parent">
-    <joint name="laser" type="fixed">
-      <origin xyz="0.15 0.0 0.360" rpy="3.14159 0.0 0.0" />
-      <parent link="base_link" />
-      <child link="base_laser_link" />
-    </joint>
-    <link name="base_laser_link">
-      <visual>
-        <geometry>
-          <box size="0.00 0.05 0.06" />
-        </geometry>
-        <material name="Green" />
-      </visual>
-      <inertial>
-        <mass value="0.000001" />
-        <origin xyz="0 0 0" />
-        <inertia ixx="0.0001" ixy="0.0" ixz="0.0"
-          iyy="0.0001" iyz="0.0"
-          izz="0.0001" />
-      </inertial>
-    </link>
-    <!-- Set up laser gazebo details -->
-    <hokuyo_laser />
-  </xacro:macro>
+<robot name="sensor_rplidar" xmlns:xacro="http://ros.org/wiki/xacro">
+	<!-- Joints and Links, standard URDF stuff -->
+	<link name="rplidar_link">
+		<collision>
+			<origin xyz="0 0 0" rpy="0 0 0"/>
+			<geometry>
+				<box size="0.1 0.1 0.1"/>
+			</geometry>
+		</collision>
+		<vision>
+			<origin xyz="0 0 -0.03125" rpy="1.5707 0 0"/>
+			<geometry>
+				<box size="0.1 0.1 0.1"/>
+				<meshfile name="$(find first_robot_gazebo)/meshes/rplidar.dae" scale="0.001 0.001 0.001" />
+			</geometry>
+		</vision>
+		<inertial>
+			<mass value="1e-5"/>
+			<origin xyz="0 0 0" rpy="0 0 0"/>
+			<inertia ixx="1e-6" ixy="0" ixz="0" iyy="1e-6" iyz="0" izz="1e-6"/>
+		</inertial>
+	</link>
+	<joint name="rplidar_joint" type="fixed">
+		<axis xyz="0 1 0"/>
+		<origin xyz="0 0 0.035" rpy="0 0 0 "/>
+		<parent link="plate_top_link"/>
+		<child link="rplidar_link"/>
+	</joint>
+<gazebo reference="rplidar_link">
+	<sensor type="gpu_ray" name="head_rplidar_sensor">
+		<pose>0 0 0 0 0 0</pose>
+		<visualize>true</visualize>
+		<update_rate>10</update_rate>
+		<ray>
+			<scan>
+				<horizontal>
+					<samples>400</samples>
+					<resolution>1</resolution>
+					<min_angle>-3.14159</min_angle>
+					<max_angle>3.14159</max_angle>
+				</horizontal>
+			</scan>
+			<range>
+				<min>0.15</min>
+				<max>6.0</max>
+				<resolution>0.01</resolution>
+			</range>
+			<noise>
+				<type>gaussian</type>
+				<mean>0.0</mean>
+				<stddev>0.01</stddev>
+			</noise>
+		</ray>
+		<plugin name="gazebo_ros_head_rplidar_controller" filename="libgazebo_ros_gpu_laser.so">
+			<topicName>/scan</topicName>
+			<frameName>rplidar_link</frameName>
+		</plugin>
+	</sensor>
+</gazebo>
 </robot>

Commit message: [laser.urdf]changes added

File: sim/first_robot_gazebo/definition/laser.urdf.xacro (robot description, xacro)
@@ -2,4 +2,5 @@
 	<!-- Joints and Links, standard URDF stuff -->
 	<link name="rplidar_link">
+		<parent link="base_link"/>
 		<collision>
 			<origin xyz="0 0 0" rpy="0 0 0"/>
@@ -23,6 +24,6 @@
 	<joint name="rplidar_joint" type="fixed">
 		<axis xyz="0 1 0"/>
-		<origin xyz="0 0 0.035" rpy="0 0 0 "/>
-		<parent link="plate_top_link"/>
+		<origin xyz="0 0 0.4" rpy="0 0 0 "/>
+		<parent link="base_footprint"/>
 		<child link="rplidar_link"/>
 	</joint>

Commit message: [point transformation]new package added

File: sim/first_robot_gazebo/definition/laser.urdf.xacro (robot description, xacro)
@@ -2,5 +2,4 @@
 	<!-- Joints and Links, standard URDF stuff -->
 	<link name="rplidar_link">
-		<parent link="base_link"/>
 		<collision>
 			<origin xyz="0 0 0" rpy="0 0 0"/>
@@ -24,6 +23,6 @@
 	<joint name="rplidar_joint" type="fixed">
 		<axis xyz="0 1 0"/>
-		<origin xyz="0 0 0.4" rpy="0 0 0 "/>
-		<parent link="base_footprint"/>
+		<origin xyz="0 0 0.035" rpy="0 0 0 "/>
+		<parent link="plate_top_link"/>
 		<child link="rplidar_link"/>
 	</joint>

Commit message: [first_robot_gazebo]rplidar added

File: sim/first_robot_gazebo/definition/laser.urdf.xacro (robot description, xacro)
@@ -23,6 +23,6 @@
 	<joint name="rplidar_joint" type="fixed">
 		<axis xyz="0 1 0"/>
-		<origin xyz="0 0 0.035" rpy="0 0 0 "/>
-		<parent link="plate_top_link"/>
+		<origin xyz="0 0 0.35" rpy="0 0 0 "/>
+		<parent link="base_link"/>
 		<child link="rplidar_link"/>
 	</joint>
